File: SK9822-LedStrip/LEDStrip-SK9822.kicad_pcb (KiCad board)
At the start: 2 copper layers, 229.9 x 73.7 mm, 72 parts, among them J1 Conn_01x04, J2 Conn_01x04

Commit message: Connecting pads on SK9822 and changing edge cut to better hold footprints
Parts:
- removed D41, D42, D43, D44, D45, D46, D47, D48, D49, D50, D51, D52, D53, D54, D55, D56, D57, D58, D59, D60: APA102-2020, LED_SMD:LED-APA102-2020
- removed G*** (x2): LOGO, BikeLights:SkullSmall
- removed REF (x6): Fiducial_0.75mm_Mask1.5mm, Fiducial:Fiducial_0.75mm_Mask1.5mm
- D1, D10, D11, D12, D13, D14, D15, D16, D17, D18, D19, D2, D20, D21, D22, D23, D24, D25, D26, D27, D28, D29, D3, D30, D31, D32, D33, D34, D35, D36, D37, D38, D39, D4, D40, D5, D6, D7, D8, D9: value APA102-2020 -> SK9822; footprint LED_SMD:LED-APA102-2020 -> SK9822:SK9822
- J1, J2: value Conn_01x04 -> TE_1-1123723-4
- moved D35 98.1 mm to (248.9, 90.4)
- moved D34 95.3 mm to (242.3, 90.4)
- moved D33 92.5 mm to (235.7, 90.4)
- moved D32 89.7 mm to (229.1, 90.4)
- moved D31 86.9 mm to (222.5, 90.4)
- moved D30 84.1 mm to (215.9, 90.4)
- moved D29 81.3 mm to (209.3, 90.4)
- moved D28 78.5 mm to (202.7, 90.4)
- moved D27 75.7 mm to (196.1, 90.4)
- moved D26 72.9 mm to (189.5, 90.4)
- moved D25 70.1 mm to (182.9, 90.4)
- moved D24 67.3 mm to (176.3, 90.4)
- moved D23 64.5 mm to (169.7, 90.4)
- moved D22 61.7 mm to (163.1, 90.4)
- moved D21 58.9 mm to (156.5, 90.4)
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Connections:
- D1 pad 1: /VDD -> /SDIN
- D1 pad 2: Net-(D1-Pad2) -> /CKIN
- D1 pad 3: Net-(D1-Pad3) -> /GND
- D1 pad 4: /SDIN -> /VDD
- D1 pad 5: /CKIN -> Net-(D1-Pad5)
- D1 pad 6: /GND -> Net-(D1-Pad6)
- D10 pad 1: /VDD -> Net-(D10-Pad1)
- D10 pad 3: Net-(D10-Pad3) -> /GND
- D10 pad 4: Net-(D10-Pad4) -> /VDD
- D10 pad 6: /GND -> Net-(D10-Pad6)
- D11 pad 1: /VDD -> Net-(D10-Pad6)
- D11 pad 2: Net-(D11-Pad2) -> Net-(D10-Pad5)
- D11 pad 3: Net-(D11-Pad3) -> /GND
- D11 pad 4: Net-(D10-Pad3) -> /VDD
- D11 pad 5: Net-(D10-Pad2) -> Net-(D11-Pad5)
- D11 pad 6: /GND -> Net-(D11-Pad6)
- D12 pad 1: /VDD -> Net-(D11-Pad6)
- D12 pad 2: Net-(D12-Pad2) -> Net-(D11-Pad5)
- D12 pad 3: Net-(D12-Pad3) -> /GND
- D12 pad 4: Net-(D11-Pad3) -> /VDD
- D12 pad 5: Net-(D11-Pad2) -> Net-(D12-Pad5)
- D12 pad 6: /GND -> Net-(D12-Pad6)
- D13 pad 1: /VDD -> Net-(D12-Pad6)
- D13 pad 2: Net-(D13-Pad2) -> Net-(D12-Pad5)
- D13 pad 3: Net-(D13-Pad3) -> /GND
- D13 pad 4: Net-(D12-Pad3) -> /VDD
- D13 pad 5: Net-(D12-Pad2) -> Net-(D13-Pad5)
- D13 pad 6: /GND -> Net-(D13-Pad6)
- D14 pad 1: /VDD -> Net-(D13-Pad6)
- D14 pad 2: Net-(D14-Pad2) -> Net-(D13-Pad5)
- D14 pad 3: Net-(D14-Pad3) -> /GND
- D14 pad 4: Net-(D13-Pad3) -> /VDD
- D14 pad 5: Net-(D13-Pad2) -> Net-(D14-Pad5)
- D14 pad 6: /GND -> Net-(D14-Pad6)
- D15 pad 1: /VDD -> Net-(D14-Pad6)
- D15 pad 2: Net-(D15-Pad2) -> Net-(D14-Pad5)
- D15 pad 3: Net-(D15-Pad3) -> /GND
- D15 pad 4: Net-(D14-Pad3) -> /VDD
- D15 pad 5: Net-(D14-Pad2) -> Net-(D15-Pad5)
- D15 pad 6: /GND -> Net-(D15-Pad6)
- D16 pad 1: /VDD -> Net-(D15-Pad6)
- D16 pad 2: Net-(D16-Pad2) -> Net-(D15-Pad5)
- D16 pad 3: Net-(D16-Pad3) -> /GND
- D16 pad 4: Net-(D15-Pad3) -> /VDD
- D16 pad 5: Net-(D15-Pad2) -> Net-(D16-Pad5)
- D16 pad 6: /GND -> Net-(D16-Pad6)
- D17 pad 1: /VDD -> Net-(D16-Pad6)
- D17 pad 2: Net-(D17-Pad2) -> Net-(D16-Pad5)
- D17 pad 3: Net-(D17-Pad3) -> /GND
- D17 pad 4: Net-(D16-Pad3) -> /VDD
- D17 pad 5: Net-(D16-Pad2) -> Net-(D17-Pad5)
- D17 pad 6: /GND -> Net-(D17-Pad6)
- D18 pad 1: /VDD -> Net-(D17-Pad6)
- D18 pad 2: Net-(D18-Pad2) -> Net-(D17-Pad5)
- D18 pad 3: Net-(D18-Pad3) -> /GND
- D18 pad 4: Net-(D17-Pad3) -> /VDD
- D18 pad 5: Net-(D17-Pad2) -> Net-(D18-Pad5)
- D18 pad 6: /GND -> Net-(D18-Pad6)
- D19 pad 1: /VDD -> Net-(D18-Pad6)
- D19 pad 2: Net-(D19-Pad2) -> Net-(D18-Pad5)
- D19 pad 3: Net-(D19-Pad3) -> /GND
- D19 pad 4: Net-(D18-Pad3) -> /VDD
- D19 pad 5: Net-(D18-Pad2) -> Net-(D19-Pad5)
- D19 pad 6: /GND -> Net-(D19-Pad6)
- D2 pad 1: /VDD -> Net-(D1-Pad6)
- D2 pad 2: Net-(D2-Pad2) -> Net-(D1-Pad5)
- D2 pad 3: Net-(D2-Pad3) -> /GND
- D2 pad 4: Net-(D1-Pad3) -> /VDD
- D2 pad 5: Net-(D1-Pad2) -> Net-(D2-Pad5)
- D2 pad 6: /GND -> Net-(D2-Pad6)
- D20 pad 1: /VDD -> Net-(D19-Pad6)
- D20 pad 2: Net-(D20-Pad2) -> Net-(D19-Pad5)
- D20 pad 3: Net-(D20-Pad3) -> /GND
- D20 pad 4: Net-(D19-Pad3) -> /VDD
- D20 pad 5: Net-(D19-Pad2) -> Net-(D20-Pad5)
- D20 pad 6: /GND -> Net-(D20-Pad6)
- D21 pad 1: /VDD -> Net-(D20-Pad6)
- D21 pad 2: Net-(D21-Pad2) -> Net-(D20-Pad5)
- D21 pad 3: Net-(D21-Pad3) -> /GND
- D21 pad 4: Net-(D20-Pad3) -> /VDD
- D21 pad 5: Net-(D20-Pad2) -> Net-(D21-Pad5)
- D21 pad 6: /GND -> Net-(D21-Pad6)
- D22 pad 1: /VDD -> Net-(D21-Pad6)
- D22 pad 2: Net-(D22-Pad2) -> Net-(D21-Pad5)
- D22 pad 3: Net-(D22-Pad3) -> /GND
- D22 pad 4: Net-(D21-Pad3) -> /VDD
- D22 pad 5: Net-(D21-Pad2) -> Net-(D22-Pad5)
- D22 pad 6: /GND -> Net-(D22-Pad6)
- D23 pad 1: /VDD -> Net-(D22-Pad6)
- D23 pad 2: Net-(D23-Pad2) -> Net-(D22-Pad5)
- D23 pad 3: Net-(D23-Pad3) -> /GND
- D23 pad 4: Net-(D22-Pad3) -> /VDD
- D23 pad 5: Net-(D22-Pad2) -> Net-(D23-Pad5)
- D23 pad 6: /GND -> Net-(D23-Pad6)
- D24 pad 1: /VDD -> Net-(D23-Pad6)
- D24 pad 2: Net-(D24-Pad2) -> Net-(D23-Pad5)
- D24 pad 3: Net-(D24-Pad3) -> /GND
- D24 pad 4: Net-(D23-Pad3) -> /VDD
- D24 pad 5: Net-(D23-Pad2) -> Net-(D24-Pad5)
- D24 pad 6: /GND -> Net-(D24-Pad6)
- D25 pad 1: /VDD -> Net-(D24-Pad6)
- D25 pad 2: Net-(D25-Pad2) -> Net-(D24-Pad5)
- D25 pad 3: Net-(D25-Pad3) -> /GND
- D25 pad 4: Net-(D24-Pad3) -> /VDD
- D25 pad 5: Net-(D24-Pad2) -> Net-(D25-Pad5)
- D25 pad 6: /GND -> Net-(D25-Pad6)
- D26 pad 1: /VDD -> Net-(D25-Pad6)
- D26 pad 2: Net-(D26-Pad2) -> Net-(D25-Pad5)
- D26 pad 3: Net-(D26-Pad3) -> /GND
- D26 pad 4: Net-(D25-Pad3) -> /VDD
- D26 pad 5: Net-(D25-Pad2) -> Net-(D26-Pad5)
- D26 pad 6: /GND -> Net-(D26-Pad6)
- D27 pad 1: /VDD -> Net-(D26-Pad6)
- D27 pad 2: Net-(D27-Pad2) -> Net-(D26-Pad5)
- D27 pad 3: Net-(D27-Pad3) -> /GND
- D27 pad 4: Net-(D26-Pad3) -> /VDD
- D27 pad 5: Net-(D26-Pad2) -> Net-(D27-Pad5)
- D27 pad 6: /GND -> Net-(D27-Pad6)
- D28 pad 1: /VDD -> Net-(D27-Pad6)
- D28 pad 2: Net-(D28-Pad2) -> Net-(D27-Pad5)
- D28 pad 3: Net-(D28-Pad3) -> /GND
- D28 pad 4: Net-(D27-Pad3) -> /VDD
- D28 pad 5: Net-(D27-Pad2) -> Net-(D28-Pad5)
- D28 pad 6: /GND -> Net-(D28-Pad6)
- D29 pad 1: /VDD -> Net-(D28-Pad6)
- D29 pad 2: Net-(D29-Pad2) -> Net-(D28-Pad5)
- D29 pad 3: Net-(D29-Pad3) -> /GND
- D29 pad 4: Net-(D28-Pad3) -> /VDD
- D29 pad 5: Net-(D28-Pad2) -> Net-(D29-Pad5)
- D29 pad 6: /GND -> Net-(D29-Pad6)
- D3 pad 1: /VDD -> Net-(D2-Pad6)
- D3 pad 2: Net-(D3-Pad2) -> Net-(D2-Pad5)
- D3 pad 3: Net-(D3-Pad3) -> /GND
- D3 pad 4: Net-(D2-Pad3) -> /VDD
- D3 pad 5: Net-(D2-Pad2) -> Net-(D3-Pad5)
- D3 pad 6: /GND -> Net-(D3-Pad6)
- D30 pad 1: /VDD -> Net-(D29-Pad6)
- D30 pad 2: Net-(D30-Pad2) -> Net-(D29-Pad5)
- D30 pad 3: Net-(D30-Pad3) -> /GND
- D30 pad 4: Net-(D29-Pad3) -> /VDD
- D30 pad 5: Net-(D29-Pad2) -> Net-(D30-Pad5)
- D30 pad 6: /GND -> Net-(D30-Pad6)
- D31 pad 1: /VDD -> Net-(D30-Pad6)
- D31 pad 2: Net-(D31-Pad2) -> Net-(D30-Pad5)
- D31 pad 3: Net-(D31-Pad3) -> /GND
- D31 pad 4: Net-(D30-Pad3) -> /VDD
- D31 pad 5: Net-(D30-Pad2) -> Net-(D31-Pad5)
- D31 pad 6: /GND -> Net-(D31-Pad6)
- D32 pad 1: /VDD -> Net-(D31-Pad6)
- D32 pad 2: Net-(D32-Pad2) -> Net-(D31-Pad5)
- D32 pad 3: Net-(D32-Pad3) -> /GND
- D32 pad 4: Net-(D31-Pad3) -> /VDD
- D32 pad 5: Net-(D31-Pad2) -> Net-(D32-Pad5)
- D32 pad 6: /GND -> Net-(D32-Pad6)
- D33 pad 1: /VDD -> Net-(D32-Pad6)
- D33 pad 2: Net-(D33-Pad2) -> Net-(D32-Pad5)
- D33 pad 3: Net-(D33-Pad3) -> /GND
- D33 pad 4: Net-(D32-Pad3) -> /VDD
- D33 pad 5: Net-(D32-Pad2) -> Net-(D33-Pad5)
- D33 pad 6: /GND -> Net-(D33-Pad6)
- D34 pad 1: /VDD -> Net-(D33-Pad6)
- D34 pad 2: Net-(D34-Pad2) -> Net-(D33-Pad5)
- D34 pad 3: Net-(D34-Pad3) -> /GND
- D34 pad 4: Net-(D33-Pad3) -> /VDD
- D34 pad 5: Net-(D33-Pad2) -> Net-(D34-Pad5)
- D34 pad 6: /GND -> Net-(D34-Pad6)
- D35 pad 1: /VDD -> Net-(D34-Pad6)
- D35 pad 2: Net-(D35-Pad2) -> Net-(D34-Pad5)
- D35 pad 3: Net-(D35-Pad3) -> /GND
- D35 pad 4: Net-(D34-Pad3) -> /VDD
- D35 pad 5: Net-(D34-Pad2) -> Net-(D35-Pad5)
- D35 pad 6: /GND -> Net-(D35-Pad6)
- D36 pad 1: /VDD -> Net-(D35-Pad6)
- D36 pad 2: Net-(D36-Pad2) -> Net-(D35-Pad5)
- D36 pad 3: Net-(D36-Pad3) -> /GND
- D36 pad 4: Net-(D35-Pad3) -> /VDD
- D36 pad 5: Net-(D35-Pad2) -> Net-(D36-Pad5)
- D36 pad 6: /GND -> Net-(D36-Pad6)
- D37 pad 1: /VDD -> Net-(D36-Pad6)
- D37 pad 2: Net-(D37-Pad2) -> Net-(D36-Pad5)
- D37 pad 3: Net-(D37-Pad3) -> /GND
- D37 pad 4: Net-(D36-Pad3) -> /VDD
- D37 pad 5: Net-(D36-Pad2) -> Net-(D37-Pad5)
- D37 pad 6: /GND -> Net-(D37-Pad6)
- D38 pad 1: /VDD -> Net-(D37-Pad6)
- D38 pad 2: Net-(D38-Pad2) -> Net-(D37-Pad5)
- D38 pad 3: Net-(D38-Pad3) -> /GND
- D38 pad 4: Net-(D37-Pad3) -> /VDD
- D38 pad 5: Net-(D37-Pad2) -> Net-(D38-Pad5)
- D38 pad 6: /GND -> Net-(D38-Pad6)
- D39 pad 1: /VDD -> Net-(D38-Pad6)
- D39 pad 2: Net-(D39-Pad2) -> Net-(D38-Pad5)
- D39 pad 3: Net-(D39-Pad3) -> /GND
- D39 pad 4: Net-(D38-Pad3) -> /VDD
- D39 pad 5: Net-(D38-Pad2) -> Net-(D39-Pad5)
- D39 pad 6: /GND -> Net-(D39-Pad6)
- D4 pad 1: /VDD -> Net-(D3-Pad6)
- D4 pad 2: Net-(D4-Pad2) -> Net-(D3-Pad5)
- D4 pad 3: Net-(D4-Pad3) -> /GND
- D4 pad 4: Net-(D3-Pad3) -> /VDD
- D4 pad 5: Net-(D3-Pad2) -> Net-(D4-Pad5)
- D4 pad 6: /GND -> Net-(D4-Pad6)
- D40 pad 1: /VDD -> Net-(D39-Pad6)
- D40 pad 2: Net-(D40-Pad2) -> Net-(D39-Pad5)
- D40 pad 3: Net-(D40-Pad3) -> /GND
- D40 pad 4: Net-(D39-Pad3) -> /VDD
- D40 pad 5: Net-(D39-Pad2) -> /CKOUT
- D40 pad 6: /GND -> /SDOUT
- D5 pad 1: /VDD -> Net-(D4-Pad6)
- D5 pad 2: Net-(D5-Pad2) -> Net-(D4-Pad5)
- D5 pad 3: Net-(D5-Pad3) -> /GND
- D5 pad 4: Net-(D4-Pad3) -> /VDD
- D5 pad 5: Net-(D4-Pad2) -> Net-(D5-Pad5)
- D5 pad 6: /GND -> Net-(D5-Pad6)
- D6 pad 1: /VDD -> Net-(D5-Pad6)
- D6 pad 2: Net-(D6-Pad2) -> Net-(D5-Pad5)
- D6 pad 3: Net-(D6-Pad3) -> /GND
- D6 pad 4: Net-(D5-Pad3) -> /VDD
- D6 pad 5: Net-(D5-Pad2) -> Net-(D6-Pad5)
- D6 pad 6: /GND -> Net-(D6-Pad6)
- D7 pad 1: /VDD -> Net-(D6-Pad6)
- D7 pad 2: Net-(D7-Pad2) -> Net-(D6-Pad5)
- D7 pad 3: Net-(D7-Pad3) -> /GND
- D7 pad 4: Net-(D6-Pad3) -> /VDD
- D7 pad 5: Net-(D6-Pad2) -> Net-(D7-Pad5)
- D7 pad 6: /GND -> Net-(D7-Pad6)
- D8 pad 1: /VDD -> Net-(D7-Pad6)
- D8 pad 2: Net-(D8-Pad2) -> Net-(D7-Pad5)
- D8 pad 3: Net-(D8-Pad3) -> /GND
- D8 pad 4: Net-(D7-Pad3) -> /VDD
- D8 pad 5: Net-(D7-Pad2) -> Net-(D8-Pad5)
- D8 pad 6: /GND -> Net-(D8-Pad6)
- D9 pad 1: /VDD -> Net-(D8-Pad6)
- D9 pad 2: Net-(D10-Pad5) -> Net-(D8-Pad5)
- D9 pad 3: Net-(D10-Pad4) -> /GND
- D9 pad 4: Net-(D8-Pad3) -> /VDD
- D9 pad 5: Net-(D8-Pad2) -> Net-(D10-Pad2)
- D9 pad 6: /GND -> Net-(D10-Pad1)
Routing:
- net /VDD: track 453.1 -> 298.5 mm
- net /GND: track 143.4 -> 26.2 mm, vias 120 -> 0
- net /SDIN: track 16.1 -> 0.00 mm
- net /SDOUT: track 16.0 -> 0.00 mm
- net /CKIN: track 10.9 -> 0.00 mm
- net /CKOUT: track 10.9 -> 0.00 mm
- net Net-(D8-Pad6): track 0.00 -> 2.20 mm
- net Net-(D8-Pad5): track 0.00 -> 2.20 mm
- net Net-(D7-Pad6): track 0.00 -> 2.20 mm
- net Net-(D7-Pad5): track 0.00 -> 2.20 mm
- net Net-(D34-Pad6): track 0.00 -> 2.20 mm
- net Net-(D34-Pad5): track 0.00 -> 2.20 mm
- net Net-(D33-Pad6): track 0.00 -> 2.20 mm
- net Net-(D33-Pad5): track 0.00 -> 2.20 mm
- net Net-(D32-Pad6): track 0.00 -> 2.20 mm
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Other:
- board size 229.9 x 73.7 mm -> 231.4 x 73.7 mm

Commit message: Adding Depot 37 logo and removing wings from the middle of sk9822 pcb
Parts:
- removed D36, D37, D38, D39, D40: SK9822, SK9822:SK9822
- added G***: LOGO, lib:SkullSmall, F.Cu at (237.0, 85.3)
- added G***: LOGO, lib:SkullSmall, F.Cu at (32.0, 85.3)
- moved C2 3.84 mm to (233.9, 97.3)
- moved C1 3.56 mm to (33.5, 97.0)
Connections:
- D35 pad 5: Net-(D35-Pad5) -> /CKOUT
- D35 pad 6: Net-(D35-Pad6) -> /SDOUT
Routing:
- net /GND: track 26.2 -> 99.2 mm, vias 0 -> 34
- net /SDOUT: track 0.00 -> 17.6 mm, vias 0 -> 1
- net /SDIN: track 0.00 -> 17.4 mm, vias 0 -> 1
- net /CKIN: track 0.00 -> 14.8 mm, vias 0 -> 1
- net /CKOUT: track 0.00 -> 12.7 mm, vias 0 -> 1
Other:
- outline, holes or cut-outs redrawn
- board text added: "VDD CKIN SDIN GND"
- board text added: "VDD CKOUT SDOUT GND"

Commit message: Prepared for mounting hardware
This version has the straight mounting wings
Parts:
- moved G*** 42.3 mm to (54.1, 121.4), turned to 270 degrees
- moved D10 39.0 mm to (93.2, 128.3)
- moved D16 39.0 mm to (132.8, 128.3)
- moved D18 39.0 mm to (146.1, 128.3)
- moved D2 39.0 mm to (40.4, 128.3)
- moved D3 39.0 mm to (47.0, 128.3)
- moved D33 39.0 mm to (245.1, 128.3)
- moved D4 39.0 mm to (53.6, 128.3)
- moved D5 39.0 mm to (60.2, 128.3)
- moved D6 39.0 mm to (66.8, 128.3)
- moved D7 39.0 mm to (73.4, 128.3)
- moved D8 39.0 mm to (80.0, 128.3)
- moved D9 39.0 mm to (86.6, 128.3)
- moved J1 39.0 mm to (33.3, 135.4)
- moved D1 39.0 mm to (33.8, 128.3)
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Routing:
- net /SDIN: track 17.4 -> 18.9 mm
- net /CKIN: track 14.8 -> 13.6 mm
Other:
- board size 231.4 x 73.7 mm -> 231.4 x 145 mm
- board text added: "V1.0"

Commit message: Curved Mounting Wing
Other:
- outline, holes or cut-outs redrawn
Changed lines of the file:
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@@
     )
   )
-  (gr_text "V1.0 " (at 30.734 114.808 270) (layer F.SilkS)
+  (gr_arc (start 234.175265 42.100516) (end 247.951421 37.576411) (angle -179.9999988) (layer Edge.Cuts) (width 0.05))
+  (gr_arc (start 235.07869 44.658718) (end 241.22456 42.542525) (angle -179.9999971) (layer Edge.Cuts) (width 0.05))
+  (gr_arc (start 26.924 110.236) (end 238.588 116) (angle -19) (layer Edge.Cuts) (width 0.05))
+  (gr_arc (start 26.924 110.236) (end 251.588 116) (angle -19) (layer Edge.Cuts) (width 0.05))
+  (gr_arc (start 26.924 110.236) (end 230.588 110.236) (angle -18.2) (layer Edge.Cuts) (width 0.05))
+  (gr_arc (start 26.924 110.236) (end 259.588 110.236) (angle -18.19753673) (layer Edge.Cuts) (width 0.05))
+  (gr_text "V1.0 " (at 31.496 79.756 270) (layer F.SilkS)
     (effects (font (size 1 1) (thickness 0.15)))
   )
   (gr_line (start 72.39 125.444) (end 215.396 125.444) (layer Edge.Cuts) (width 0.05))
-  (gr_arc (start 215.396 110.252) (end 215.396 125.444) (angle -90) (layer Edge.Cuts) (width 0.05))
-  (gr_line (start 230.588 41.226) (end 230.588 110.252) (layer Edge.Cuts) (width 0.05))
-  (gr_line (start 238.588 41.226) (end 238.588 116) (layer Edge.Cuts) (width 0.05))
-  (gr_line (start 251.588 116) (end 251.588 41.226) (layer Edge.Cuts) (width 0.05))
+  (gr_arc (start 215.396 110.252) (end 215.396 125.444) (angle -90.06034308) (layer Edge.Cuts) (width 0.05))
   (gr_arc (start 245.088 116) (end 251.588 116) (angle 180) (layer Edge.Cuts) (width 0.05))
-  (gr_arc (start 245.088 41.226) (end 251.588 41.226) (angle -180) (layer Edge.Cuts) (width 0.05))
-  (gr_line (start 259.588 99.695) (end 259.588 41.226) (layer Edge.Cuts) (width 0.05))
-  (gr_arc (start 245.088 41.226) (end 259.588 41.226) (angle -180) (layer Edge.Cuts) (width 0.05))
   (gr_line (start 72.39 136.938) (end 215.396 136.938) (layer Edge.Cuts) (width 0.05))
   (gr_line (start 230.588 157.226) (end 230.588 152.13) (layer Edge.Cuts) (width 0.05))
@@
   )
   (gr_line (start 28.194 41.226) (end 28.194 144.145) (layer Edge.Cuts) (width 0.05))
-  (gr_text Depot37.net (at 32.258 90 -90) (layer F.SilkS)
+  (gr_text Depot37.net (at 32.004 110.49 -90) (layer F.SilkS)
     (effects (font (size 3 3) (thickness 0.5)))
   )
-  (gr_text Depot37.net (at 255.778 90 -90) (layer F.SilkS)
+  (gr_text Depot37.net (at 255.27 110.49 -90) (layer F.SilkS)
     (effects (font (size 3 3) (thickness 0.5)))
   )
@@
   (gr_line (start 28.194 144.145) (end 28.194 157.226) (layer Edge.Cuts) (width 0.05))
   (gr_line (start 259.588 144.145) (end 259.588 157.226) (layer Edge.Cuts) (width 0.05))
-  (gr_line (start 259.588 128.143) (end 259.588 99.695) (layer Edge.Cuts) (width 0.05))
+  (gr_line (start 259.588 128.143) (end 259.588 110.236) (layer Edge.Cuts) (width 0.05))
   (via (at 37.592 131.572) (size 0.8) (drill 0.4) (layers F.Cu B.Cu) (net 1))
   (segment (start 37.49 131.47) (end 37.592 131.572) (width 1) (layer F.Cu) (net 1))
